File: milled/bpw.sch (KiCad schematic (older format))
At the start: 8 parts, among them U1 ZXSC380

Commit message: Joule Thief
Parts:
- removed C1: 1uF, Capacitor_SMD:C_0603_1608Metric_Pad1.08x0.95mm_HandSolder, symbol Device:C
- removed D3, D4: D_Schottky, Diode_SMD:D_0603_1608Metric_Pad1.05x0.95mm_HandSolder, symbol Device:D_Schottky
- U1: symbol ml-symbols:ZXSC380 -> bpw-rescue:ZXSC380-ml-symbols
Connections:
- net labels removed: GND
- wire segments 25 -> 15
Other:
- moved on the sheet: L1
Changed lines of the file:
@@
-$EndComp
-$Comp
-L Device:C C1
-U 1 1 5FF67473
-P 4100 4300
-F 0 "C1" H 4215 4346 50  0000 L CNN
-F 1 "1uF" H 4215 4255 50  0000 L CNN
-F 2 "Capacitor_SMD:C_0603_1608Metric_Pad1.08x0.95mm_HandSolder" H 4138 4150 50  0001 C CNN
-F 3 "~" H 4100 4300 50  0001 C CNN
-	1    4100 4300
-	1    0    0    -1
 $EndComp
 $Comp
 L Device:L L1
 U 1 1 5FF67AED
-P 4300 3300
-F 0 "L1" V 4490 3300 50  0000 C CNN
-F 1 "100uH" V 4399 3300 50  0000 C CNN
-F 2 "Inductor_SMD:L_0603_1608Metric_Pad1.05x0.95mm_HandSolder" H 4300 3300 50  0001 C CNN
-F 3 "~" H 4300 3300 50  0001 C CNN
-	1    4300 3300
+P 5450 3750
+F 0 "L1" V 5640 3750 50  0000 C CNN
+F 1 "100uH" V 5549 3750 50  0000 C CNN
+F 2 "Inductor_SMD:L_0603_1608Metric_Pad1.05x0.95mm_HandSolder" H 5450 3750 50  0001 C CNN
+F 3 "~" H 5450 3750 50  0001 C CNN
+	1    5450 3750
 	0    -1   -1   0
 $EndComp
@@
 $EndComp
 $Comp
-L ml-symbols:ZXSC380 U1
+L bpw-rescue:ZXSC380-ml-symbols U1
 U 1 1 5FF6E683
 P 4950 4250
@@
 	5750 4950 5750 4700
 Wire Wire Line
-	4950 4950 4700 4950
-Wire Wire Line
 	3550 4950 3550 4650
 Connection ~ 4950 4950
 Wire Wire Line
 	3550 4300 3550 4350
-Wire Wire Line
-	4100 4450 4100 4950
-Connection ~ 4100 4950
-Wire Wire Line
-	4100 4950 3550 4950
-$Comp
-L Device:D_Schottky D3
-U 1 1 5FF6FFC0
-P 3850 3750
-F 0 "D3" H 3850 3533 50  0000 C CNN
-F 1 "D_Schottky" H 3850 3624 50  0000 C CNN
-F 2 "Diode_SMD:D_0603_1608Metric_Pad1.05x0.95mm_HandSolder" H 3850 3750 50  0001 C CNN
-F 3 "~" H 3850 3750 50  0001 C CNN
-	1    3850 3750
-	-1   0    0    1
-$EndComp
-$Comp
-L Device:D_Schottky D4
-U 1 1 5FF70BB4
-P 4950 3550
-F 0 "D4" V 4996 3470 50  0000 R CNN
-F 1 "D_Schottky" V 4905 3470 50  0000 R CNN
-F 2 "Diode_SMD:D_0603_1608Metric_Pad1.05x0.95mm_HandSolder" H 4950 3550 50  0001 C CNN
-F 3 "~" H 4950 3550 50  0001 C CNN
-	1    4950 3550
-	0    -1   -1   0
-$EndComp
-Wire Wire Line
-	4000 3750 4100 3750
 Wire Wire Line
 	4950 3750 4950 3800
@@
 Connection ~ 4950 3750
 Wire Wire Line
-	4100 4150 4100 3750
-Connection ~ 4100 3750
+	3550 3750 3550 4000
+Connection ~ 5750 4250
 Wire Wire Line
-	4100 3750 4950 3750
+	5600 3750 5750 3750
 Wire Wire Line
-	3700 3750 3550 3750
+	5750 3750 5750 4250
 Wire Wire Line
-	3550 3750 3550 4000
+	5300 3750 4950 3750
 Wire Wire Line
-	4950 3400 4950 3300
+	3550 4950 4950 4950
 Wire Wire Line
-	4950 3300 4450 3300
-Wire Wire Line
-	3550 3750 3550 3300
-Wire Wire Line
-	3550 3300 4150 3300
-Connection ~ 3550 3750
-Wire Wire Line
-	4950 3300 5750 3300
-Wire Wire Line
-	5750 3300 5750 4250
-Connection ~ 4950 3300
-Connection ~ 5750 4250
-$Comp
-L power:GND #PWR?
-U 1 1 5FF79A39
-P 4700 5000
-F 0 "#PWR?" H 4700 4750 50  0001 C CNN
-F 1 "GND" H 4705 4827 50  0000 C CNN
-F 2 "" H 4700 5000 50  0001 C CNN
-F 3 "" H 4700 5000 50  0001 C CNN
-	1    4700 5000
-	1    0    0    -1
-$EndComp
-Wire Wire Line
-	4700 4950 4700 5000
-Connection ~ 4700 4950
-Wire Wire Line
-	4700 4950 4100 4950
+	3550 3750 4950 3750
 $EndSCHEMATC
